File: schemas/DMX.sch (KiCad schematic (older format))
At the start: 8 parts, among them IC1 ATMEGA328P-P, K1 CONN_3, K2 CONN_3, P1 CONN_14, P2 CONN_14, X1 CRYSTAL

Commit message: avancement routage pcb
Parts:
- removed K1, K2: CONN_3, symbol CONN_3
- added P3: CONN_3X2, symbol CONN_3X2
Connections:
- no-connect marks 0 -> 5
Changed lines of the file:
@@
-EESchema Schematic File Version 2  date sam. 08 févr. 2014 12:46:17 CET
+EESchema Schematic File Version 2  date sam. 08 févr. 2014 16:00:57 CET
 LIBS:power
 LIBS:device
@@
 Comment4 ""
 $EndDescr
+NoConn ~ 7050 4150
+NoConn ~ 7050 4050
+NoConn ~ 7050 3950
+NoConn ~ 7050 3850
+NoConn ~ 7050 3200
+$Comp
+L CONN_3X2 P3
+U 1 1 52F6421B
+P 2650 3700
+F 0 "P3" H 2650 3950 50  0000 C CNN
+F 1 "CONN_3X2" V 2650 3750 40  0000 C CNN
+	1    2650 3700
+	1    0    0    -1
+$EndComp
 Connection ~ 19750 5100
 Wire Wire Line
@@
 	5150 4050 4900 4050
 Wire Wire Line
-	3400 3200 3150 3200
-Wire Wire Line
-	1950 3300 2200 3300
-Wire Wire Line
-	1950 3100 2200 3100
+	3300 3650 3050 3650
+Wire Wire Line
+	2000 3750 2250 3750
+Wire Wire Line
+	2000 3550 2250 3550
 Connection ~ 5000 4150
 Wire Wire Line
@@
 	5000 4250 5000 4050
 Wire Wire Line
-	2200 3200 1950 3200
-Wire Wire Line
-	3150 3300 3400 3300
-Wire Wire Line
-	3150 3100 3400 3100
+	2250 3650 2000 3650
+Wire Wire Line
+	3050 3750 3300 3750
+Wire Wire Line
+	3050 3550 3300 3550
 Connection ~ 5000 1750
 Wire Wire Line
@@
 	7400 1950 7050 1950
 Wire Wire Line
-	5150 2150 5000 2150
-Wire Wire Line
-	5000 2150 5000 1750
+	5000 2150 5150 2150
+Wire Wire Line
+	5000 1750 5000 2150
 Wire Wire Line
 	2100 1400 2100 1250
@@
 Text GLabel 4900 4050 0    60   Input ~ 0
 GND
-Text GLabel 3400 3100 2    60   Input ~ 0
+Text GLabel 3300 3550 2    60   Input ~ 0
 VCC
-Text GLabel 3400 3200 2    60   Input ~ 0
+Text GLabel 3300 3650 2    60   Input ~ 0
 MOSI
-Text GLabel 3400 3300 2    60   Input ~ 0
+Text GLabel 3300 3750 2    60   Input ~ 0
 GND
-Text GLabel 1950 3300 0    60   Input ~ 0
+Text GLabel 2000 3750 0    60   Input ~ 0
 RST
-Text GLabel 1950 3200 0    60   Input ~ 0
+Text GLabel 2000 3650 0    60   Input ~ 0
 SCK
-Text GLabel 1950 3100 0    60   Input ~ 0
+Text GLabel 2000 3550 0    60   Input ~ 0
 MISO
 $Comp
-L CONN_3 K2
-U 1 1 52F4B147
-P 2800 3200
-F 0 "K2" V 2750 3200 50  0000 C CNN
-F 1 "CONN_3" V 2850 3200 40  0000 C CNN
-	1    2800 3200
-	-1   0    0    1
-$EndComp
-$Comp
-L CONN_3 K1
-U 1 1 52F4B144
-P 2550 3200
-F 0 "K1" V 2500 3200 50  0000 C CNN
-F 1 "CONN_3" V 2600 3200 40  0000 C CNN
-	1    2550 3200
-	1    0    0    -1
-$EndComp
-$Comp
 L GND #PWR01

Commit message: agencement PIN différent pour essayer d'avoir moins de Strap, Reste un Pb de Plan de masse à corriger
Parts:
- added 10k: R, symbol R
Connections:
- no-connect marks 5 -> 0
Changed lines of the file:
@@
-EESchema Schematic File Version 2  date sam. 08 févr. 2014 16:00:57 CET
+EESchema Schematic File Version 2  date dim. 09 févr. 2014 23:20:03 CET
 LIBS:power
 LIBS:device
@@
 LIBS:contrib
 LIBS:valves
+LIBS:DMX-cache
 EELAYER 25  0
 EELAYER END
@@
 Sheet 1 1
 Title ""
-Date "8 feb 2014"
+Date "9 feb 2014"
 Rev ""
 Comp ""
@@
 Comment4 ""
 $EndDescr
-NoConn ~ 7050 4150
-NoConn ~ 7050 4050
-NoConn ~ 7050 3950
-NoConn ~ 7050 3850
-NoConn ~ 7050 3200
+Text GLabel 4500 2150 0    60   Input ~ 0
+RST
+$Comp
+L R 10k
+U 1 1 52F7FEDE
+P 4750 2150
+F 0 "10k" V 4830 2150 50  0000 C CNN
+F 1 "R" V 4750 2150 50  0000 C CNN
+	1    4750 2150
+	0    -1   -1   0
+$EndComp
+Connection ~ 7300 2250
+Wire Wire Line
+	7300 1750 7300 2250
+Wire Wire Line
+	7550 3450 7050 3450
+Wire Wire Line
+	7550 3200 7050 3200
+Wire Wire Line
+	7550 3000 7050 3000
+Wire Wire Line
+	7550 2800 7050 2800
+Wire Wire Line
+	7550 2550 7050 2550
+Wire Wire Line
+	7050 2350 7550 2350
+Wire Wire Line
+	7550 2050 7050 2050
+Wire Wire Line
+	7550 2150 7050 2150
+Connection ~ 19750 5100
+Wire Wire Line
+	3300 2350 3300 2500
+Wire Wire Line
+	3100 2350 3100 2500
+Wire Wire Line
+	2900 2350 2900 2500
+Wire Wire Line
+	2700 2350 2700 2500
+Wire Wire Line
+	2500 2350 2500 2500
+Wire Wire Line
+	2300 2350 2300 2500
+Wire Wire Line
+	2200 1250 2200 1400
+Wire Wire Line
+	5150 1850 4900 1850
+Connection ~ 5000 4050
+Wire Wire Line
+	5150 4050 4900 4050
+Wire Wire Line
+	3300 3650 3050 3650
+Wire Wire Line
+	2000 3750 2250 3750
+Wire Wire Line
+	2000 3550 2250 3550
+Connection ~ 5000 4150
+Wire Wire Line
+	5150 4150 5000 4150
+Connection ~ 9300 2200
+Wire Wire Line
+	9300 2450 9300 2200
+Wire Wire Line
+	8900 1450 8900 1800
+Wire Wire Line
+	8900 1800 9000 1800
+Wire Wire Line
+	9600 1800 9700 1800
+Wire Wire Line
+	8900 2200 9700 2200
+Wire Wire Line
+	9700 1800 9700 1450
+Wire Wire Line
+	5000 4050 5000 4250
+Wire Wire Line
+	2250 3650 2000 3650
+Wire Wire Line
+	3050 3750 3300 3750
+Wire Wire Line
+	3050 3550 3300 3550
+Connection ~ 5000 1750
+Connection ~ 5000 1850
+Wire Wire Line
+	5150 2150 5000 2150
+Wire Wire Line
+	5000 2150 5000 1750
+Wire Wire Line
+	2100 1400 2100 1250
+Wire Wire Line
+	3000 1250 3000 1400
+Wire Wire Line
+	2400 2350 2400 2500
+Wire Wire Line
+	2600 2350 2600 2500
+Wire Wire Line
+	2800 2350 2800 2500
+Wire Wire Line
+	3000 2350 3000 2500
+Wire Wire Line
+	3200 2350 3200 2500
+Wire Wire Line
+	7550 1950 7050 1950
+Wire Wire Line
+	7050 2250 7550 2250
+Wire Wire Line
+	7550 2450 7050 2450
+Wire Wire Line
+	7550 2700 7050 2700
+Wire Wire Line
+	7050 2900 7550 2900
+Wire Wire Line
+	7050 3100 7550 3100
+Wire Wire Line
+	7050 3300 7550 3300
+Wire Wire Line
+	7200 1750 7200 2150
+Connection ~ 7200 2150
+Wire Wire Line
+	7400 1750 7400 2350
+Connection ~ 7400 2350
 $Comp
 L CONN_3X2 P3
@@
 	1    0    0    -1
 $EndComp
-Connection ~ 19750 5100
-Wire Wire Line
-	7400 3750 7050 3750
-Wire Wire Line
-	7400 3550 7050 3550
-Wire Wire Line
-	7400 3000 7050 3000
-Wire Wire Line
-	7400 2800 7050 2800
-Wire Wire Line
-	3300 2350 3300 2500
-Wire Wire Line
-	3100 2350 3100 2500
-Wire Wire Line
-	2900 2350 2900 2500
-Wire Wire Line
-	2700 2350 2700 2500
-Wire Wire Line
-	2500 2350 2500 2500
-Wire Wire Line
-	2300 2350 2300 2500
-Wire Wire Line
-	2200 1250 2200 1400
-Wire Wire Line
-	7400 3450 7050 3450
-Wire Wire Line
-	7400 2050 7050 2050
-Connection ~ 7250 2150
-Wire Wire Line
-	7250 1550 7250 2150
-Wire Wire Line
-	5150 1850 4900 1850
-Wire Wire Line
-	7400 2250 7050 2250
-Wire Wire Line
-	7400 3300 7050 3300
-Connection ~ 5000 4050
-Wire Wire Line
-	5150 4050 4900 4050
-Wire Wire Line
-	3300 3650 3050 3650
-Wire Wire Line
-	2000 3750 2250 3750
-Wire Wire Line
-	2000 3550 2250 3550
-Connection ~ 5000 4150
-Wire Wire Line
-	5150 4150 5000 4150
-Connection ~ 9300 2200
-Wire Wire Line
-	9300 2450 9300 2200
-Wire Wire Line
-	8900 1450 8900 1800
-Wire Wire Line
-	7050 2450 7400 2450
-Wire Wire Line
-	8900 1800 9000 1800
-Wire Wire Line
-	9600 1800 9700 1800
-Wire Wire Line
-	8900 2200 9700 2200
-Wire Wire Line
-	7050 2550 7400 2550
-Wire Wire Line
-	9700 1800 9700 1450
-Wire Wire Line
-	5000 4250 5000 4050
-Wire Wire Line
-	2250 3650 2000 3650
-Wire Wire Line
-	3050 3750 3300 3750
-Wire Wire Line
-	3050 3550 3300 3550
-Connection ~ 5000 1750
-Wire Wire Line
-	7050 2350 7400 2350
-Wire Wire Line
-	7400 2150 7050 2150
-Connection ~ 5000 1850
-Wire Wire Line
-	7400 1950 7050 1950
-Wire Wire Line
-	5000 2150 5150 2150
-Wire Wire Line
-	5000 1750 5000 2150
-Wire Wire Line
-	2100 1400 2100 1250
-Wire Wire Line
-	3000 1250 3000 1400
-Wire Wire Line
-	2400 2350 2400 2500
-Wire Wire Line
-	2600 2350 2600 2500
-Wire Wire Line
-	2800 2350 2800 2500
-Wire Wire Line
-	3000 2350 3000 2500
-Wire Wire Line
-	3200 2350 3200 2500
-Wire Wire Line
-	7050 2700 7400 2700
-Wire Wire Line
-	7400 2900 7050 2900
-Wire Wire Line
-	7400 3100 7050 3100
-Wire Wire Line
-	7400 3650 7050 3650
-Text GLabel 7400 3750 2    60   Input ~ 0
+Text GLabel 7550 1950 2    60   Input ~ 0
 s8
-Text GLabel 7400 3650 2    60   Input ~ 0
+Text GLabel 7550 2050 2    60   Input ~ 0
 s7
-Text GLabel 7400 3100 2    60   Input ~ 0
+Text GLabel 7550 2350 2    60   Input ~ 0
 s5
-Text GLabel 7400 3000 2    60   Input ~ 0
+Text GLabel 7550 2700 2    60   Input ~ 0
 s4
-Text GLabel 7400 2900 2    60   Input ~ 0
+Text GLabel 7550 2800 2    60   Input ~ 0
 s3
-Text GLabel 7400 2800 2    60   Input ~ 0
+Text GLabel 7550 2900 2    60   Input ~ 0
 s2
-Text GLabel 7400 2700 2    60   Input ~ 0
+Text GLabel 7550 3000 2    60   Input ~ 0
 s1
-Text GLabel 7400 3550 2    60   Input ~ 0
+Text GLabel 7550 2250 2    60   Input ~ 0
 s6
 Text GLabel 3000 1400 3    60   Output ~ 0
 s6
+Text GLabel 3100 2500 3    60   Output ~ 0
+PWM3
 Text GLabel 2200 1400 3    60   Output ~ 0
-PWM3
-Text GLabel 2100 1400 3    60   Output ~ 0
 PWM2
 Entry Wire Line
@@
 Text GLabel 3200 2500 3    60   Output ~ 0
 s7
-Text GLabel 3100 2500 3    60   Output ~ 0
+Text GLabel 2100 1400 3    60   Output ~ 0
 PWM1
 Text GLabel 3000 2500 3    60   Output ~ 0
@@
 Text GLabel 2300 2500 3    60   Output ~ 0
 RX
-Text GLabel 7400 3450 2    60   Input ~ 0
+Text GLabel 7550 3450 2    60   Input ~ 0
 RX
-Text GLabel 7250 1550 1    60   Input ~ 0
+Text GLabel 7550 2150 2    60   Input ~ 0
 PWM3
-Text GLabel 7400 2050 2    60   Input ~ 0
+Text GLabel 7550 3100 2    60   Input ~ 0
 PWM2
-Text GLabel 7400 1950 2    60   Input ~ 0
+Text GLabel 7550 3200 2    60   Input ~ 0
 PWM1
-Text GLabel 7400 3300 2    60   Input ~ 0
+Text GLabel 7550 3300 2    60   Input ~ 0
 RST
-Text GLabel 7400 2350 2    60   Input ~ 0
+Text GLabel 7400 1750 1    60   Input ~ 0
 SCK
-Text GLabel 7400 2250 2    60   Input ~ 0
+Text GLabel 7300 1750 1    60   Input ~ 0
 MISO
-Text GLabel 7400 2150 2    60   Input ~ 0
+Text GLabel 7200 1750 1    60   Input ~ 0
 MOSI
 Text GLabel 4900 1850 0    60   Input ~ 0
@@
 	1    0    0    -1
 $EndComp
-Text GLabel 7400 2550 2    60   Input ~ 0
+Text GLabel 7550 2550 2    60   Input ~ 0
 xtl2
-Text GLabel 7400 2450 2    60   Input ~ 0
+Text GLabel 7550 2450 2    60   Input ~ 0
 xtl1
 Text GLabel 9700 1450 1    60   Input ~ 0

Commit message: on approche la perfection
Parts:
- renumbered 10k to 10k1
Connections:
- wire segments 50 -> 46
Changed lines of the file:
@@
-EESchema Schematic File Version 2  date dim. 09 févr. 2014 23:20:03 CET
+EESchema Schematic File Version 2  date lun. 10 févr. 2014 23:25:53 CET
 LIBS:power
 LIBS:device
@@
 Sheet 1 1
 Title ""
-Date "9 feb 2014"
+Date "10 feb 2014"
 Rev ""
 Comp ""
@@
 Comment4 ""
 $EndDescr
+Wire Wire Line
+	7050 4150 7400 4150
+Wire Wire Line
+	7300 1750 7300 2250
+Wire Wire Line
+	7400 4050 7050 4050
+Connection ~ 7200 2150
+Wire Wire Line
+	7550 2150 7050 2150
+Wire Wire Line
+	7050 3300 7050 3300
+Wire Wire Line
+	7550 2450 7050 2450
+Wire Wire Line
+	7550 2050 7050 2050
+Wire Wire Line
+	7050 1850 7550 1850
+Wire Wire Line
+	3200 2350 3200 2500
+Wire Wire Line
+	3000 2350 3000 2500
+Wire Wire Line
+	2800 2350 2800 2500
+Wire Wire Line
+	2600 2350 2600 2500
+Wire Wire Line
+	2400 2350 2400 2500
+Wire Wire Line
+	3000 1250 3000 1400
+Wire Wire Line
+	2100 1400 2100 1250
+Wire Wire Line
+	5000 1750 5000 2150
+Wire Wire Line
+	5000 2150 5150 2150
+Connection ~ 5000 1850
+Connection ~ 5000 1750
+Wire Wire Line
+	3050 3550 3300 3550
+Wire Wire Line
+	3050 3750 3300 3750
+Wire Wire Line
+	2250 3650 2000 3650
+Wire Wire Line
+	5000 4250 5000 4050
+Wire Wire Line
+	9700 1450 9700 1800
+Wire Wire Line
+	9700 2200 8900 2200
+Wire Wire Line
+	9700 1800 9600 1800
+Wire Wire Line
+	9000 1800 8900 1800
+Wire Wire Line
+	8900 1800 8900 1450
+Wire Wire Line
+	9300 2450 9300 2200
+Connection ~ 9300 2200
+Wire Wire Line
+	5150 4150 5000 4150
+Connection ~ 5000 4150
+Wire Wire Line
+	2000 3550 2250 3550
+Wire Wire Line
+	2000 3750 2250 3750
+Wire Wire Line
+	3300 3650 3050 3650
+Wire Wire Line
+	4900 4050 5150 4050
+Connection ~ 5000 4050
+Wire Wire Line
+	4900 1850 5150 1850
+Wire Wire Line
+	2200 1250 2200 1400
+Wire Wire Line
+	2300 2350 2300 2500
+Wire Wire Line
+	2500 2350 2500 2500
+Wire Wire Line
+	2700 2350 2700 2500
+Wire Wire Line
+	2900 2350 2900 2500
+Wire Wire Line
+	3100 2350 3100 2500
+Wire Wire Line
+	3300 2350 3300 2500
+Connection ~ 19750 5100
+Wire Wire Line
+	7050 2350 7550 2350
+Wire Wire Line
+	7050 2550 7550 2550
+Connection ~ 7400 2350
+Wire Wire Line
+	7550 2250 7050 2250
+Connection ~ 7300 2250
+Wire Wire Line
+	7050 3950 7400 3950
+Wire Wire Line
+	7200 1750 7200 2150
+Wire Wire Line
+	7400 2350 7400 1750
 Text GLabel 4500 2150 0    60   Input ~ 0
 RST
 $Comp
-L R 10k
+L R 10k1
 U 1 1 52F7FEDE
 P 4750 2150
-F 0 "10k" V 4830 2150 50  0000 C CNN
+F 0 "10k1" V 4830 2150 50  0000 C CNN
 F 1 "R" V 4750 2150 50  0000 C CNN
 	1    4750 2150
 	0    -1   -1   0
 $EndComp
-Connection ~ 7300 2250
-Wire Wire Line
-	7300 1750 7300 2250
-Wire Wire Line
-	7550 3450 7050 3450
-Wire Wire Line
-	7550 3200 7050 3200
-Wire Wire Line
-	7550 3000 7050 3000
-Wire Wire Line
-	7550 2800 7050 2800
-Wire Wire Line
-	7550 2550 7050 2550
-Wire Wire Line
-	7050 2350 7550 2350
-Wire Wire Line
-	7550 2050 7050 2050
-Wire Wire Line
-	7550 2150 7050 2150
-Connection ~ 19750 5100
-Wire Wire Line
-	3300 2350 3300 2500
-Wire Wire Line
-	3100 2350 3100 2500
-Wire Wire Line
-	2900 2350 2900 2500
-Wire Wire Line
-	2700 2350 2700 2500
-Wire Wire Line
-	2500 2350 2500 2500
-Wire Wire Line
-	2300 2350 2300 2500
-Wire Wire Line
-	2200 1250 2200 1400
-Wire Wire Line
-	5150 1850 4900 1850
-Connection ~ 5000 4050
-Wire Wire Line
-	5150 4050 4900 4050
-Wire Wire Line
-	3300 3650 3050 3650
-Wire Wire Line
-	2000 3750 2250 3750
-Wire Wire Line
-	2000 3550 2250 3550
-Connection ~ 5000 4150
-Wire Wire Line
-	5150 4150 5000 4150
-Connection ~ 9300 2200
-Wire Wire Line
-	9300 2450 9300 2200
-Wire Wire Line
-	8900 1450 8900 1800
-Wire Wire Line
-	8900 1800 9000 1800
-Wire Wire Line
-	9600 1800 9700 1800
-Wire Wire Line
-	8900 2200 9700 2200
-Wire Wire Line
-	9700 1800 9700 1450
-Wire Wire Line
-	5000 4050 5000 4250
-Wire Wire Line
-	2250 3650 2000 3650
-Wire Wire Line
-	3050 3750 3300 3750
-Wire Wire Line
-	3050 3550 3300 3550
-Connection ~ 5000 1750
-Connection ~ 5000 1850
-Wire Wire Line
-	5150 2150 5000 2150
-Wire Wire Line
-	5000 2150 5000 1750
-Wire Wire Line
-	2100 1400 2100 1250
-Wire Wire Line
-	3000 1250 3000 1400
-Wire Wire Line
-	2400 2350 2400 2500
-Wire Wire Line
-	2600 2350 2600 2500
-Wire Wire Line
-	2800 2350 2800 2500
-Wire Wire Line
-	3000 2350 3000 2500
-Wire Wire Line
-	3200 2350 3200 2500
-Wire Wire Line
-	7550 1950 7050 1950
-Wire Wire Line
-	7050 2250 7550 2250
-Wire Wire Line
-	7550 2450 7050 2450
-Wire Wire Line
-	7550 2700 7050 2700
-Wire Wire Line
-	7050 2900 7550 2900
-Wire Wire Line
-	7050 3100 7550 3100
-Wire Wire Line
-	7050 3300 7550 3300
-Wire Wire Line
-	7200 1750 7200 2150
-Connection ~ 7200 2150
-Wire Wire Line
-	7400 1750 7400 2350
-Connection ~ 7400 2350
 $Comp
 L CONN_3X2 P3
@@
 	1    0    0    -1
 $EndComp
-Text GLabel 7550 1950 2    60   Input ~ 0
+Text GLabel 7550 1850 2    60   Input ~ 0
 s8
 Text GLabel 7550 2050 2    60   Input ~ 0
 s7
-Text GLabel 7550 2350 2    60   Input ~ 0
+Text GLabel 7550 2150 2    60   Input ~ 0
 s5
-Text GLabel 7550 2700 2    60   Input ~ 0
+Text GLabel 7550 2250 2    60   Input ~ 0
 s4
-Text GLabel 7550 2800 2    60   Input ~ 0
+Text GLabel 7400 3950 2    60   Input ~ 0
 s3
-Text GLabel 7550 2900 2    60   Input ~ 0
+Text GLabel 7050 3850 2    60   Input ~ 0
 s2
-Text GLabel 7550 3000 2    60   Input ~ 0
+Text GLabel 7050 3750 2    60   Input ~ 0
 s1
-Text GLabel 7550 2250 2    60   Input ~ 0
+Text GLabel 7400 4050 2    60   Input ~ 0
 s6
 Text GLabel 3000 1400 3    60   Output ~ 0
@@
 Text GLabel 2300 2500 3    60   Output ~ 0
 RX
-Text GLabel 7550 3450 2    60   Input ~ 0
+Text GLabel 7050 3450 2    60   Input ~ 0
 RX
-Text GLabel 7550 2150 2    60   Input ~ 0
+Text GLabel 7400 4150 2    60   Input ~ 0
 PWM3
-Text GLabel 7550 3100 2    60   Input ~ 0
+Text GLabel 7050 3650 2    60   Input ~ 0
 PWM2
-Text GLabel 7550 3200 2    60   Input ~ 0
+Text GLabel 7050 3550 2    60   Input ~ 0
 PWM1
-Text GLabel 7550 3300 2    60   Input ~ 0
+Text GLabel 7050 3300 2    60   Input ~ 0
 RST
 Text GLabel 7400 1750 1    60   Input ~ 0
@@
 F 1 "CRYSTAL" H 9300 1650 60  0000 C CNN
 	1    9300 1800
-	1    0    0    -1
-$EndComp
-$Comp
+	1    0    0    1
+$EndComp
+$Comp
